File: misc.sch (KiCad schematic (older format))
At the start: 11 parts, among them J11 USB_OTG, U3 LP5900SDX-2.8, U4 AP7313-30SAG

Commit message: fix ldo ap7313 bug
Parts:
- U4: footprint TO_SOT_Packages_SMD:SOT-89-3 -> TO_SOT_Packages_SMD:SOT-23
Changed lines of the file:
@@
 F 0 "U4" H 6600 2675 50  0000 L CNN
 F 1 "AP7313-30SAG" H 6800 2675 50  0000 L CNN
-F 2 "TO_SOT_Packages_SMD:SOT-89-3" H 6800 2775 50  0001 C CNN
+F 2 "TO_SOT_Packages_SMD:SOT-23" H 6800 2775 50  0001 C CNN
 F 3 "" H 6800 2550 50  0001 C CNN
 	1    6800 2550
